Commit message: Negated URDF axes to make rotation convention consistent with lectures

File: reacher/data/pupper_arm.urdf (robot description, URDF)
Before this commit: robot pupper_arm, 5 links, 4 joints
Joints:
- joint baseMotor: axis 0 -1.0 0 -> 0 1 0
- joint leftFrontLowerLegMotor: axis -1.0 0 0 -> 1.0 0 0
- joint leftFrontUpperLegMotor: axis 1.0 0 0 -> -1.0 0 0

Commit message: Updated URDF to use the lengthened leg components

File: reacher/data/pupper_arm.urdf (robot description, URDF)
Before this commit: robot pupper_arm, 5 links, 4 joints
Links:
- link leftFrontLowerLeg: geometry collision box size=0.00951 0.012 0.10758; visual mesh filename=meshes/Lengthened_Lower_Leg_L.stl scale=0.001 0.001 0.001
- link leftFrontUpperLeg: geometry collision cylinder length=0.065 radius=0.015; visual mesh filename=meshes/Lengthened_Upper_Leg.stl scale=0.001 0.001 0.001
Joints:
- joint leftFrontLowerLegMotor: origin xyz=-0.004 0 -0.08 rpy=0 0 3.14159 -> xyz=-0.004 0 -0.10 rpy=0 0 3.14159
- joint leftFrontToe: origin xyz=0.002 0 -0.11 rpy=0 0 -3.14159 -> xyz=0.002 0 -0.13 rpy=0 0 -3.14159
